File: pcb/base_module/rx_mod.brd (EAGLE design)
At the start: 42.5 x 28.8 mm, 28 parts, among them U1 ATMEGA328

Commit message: base module v4.0
Parts:
- removed C2: 470uf, SparkFun-Passives:EIA7343
- removed R_RSSI: 100K, SparkFun:0603-RES
- added IC1: OPA336N, burr-brown:SOT23-5
- added R_RSSI_A: 100K, SparkFun:0603-RES
- added SJ1: (no value), jumper:SJ
- moved R_VIDOUT 0.74 mm to (19.5, 5.68)
- renumbered R_RSSI1 to R_RSSI_B
Connections:
- new net RSSI_A_FIL: IC1.1, IC1.4, SJ1.2, U1.25
- net 5V: now also IC1.5
- net GND: now also IC1.2, R_RSSI_A.1; no longer R_RSSI.1
- net N$6: no longer C2.A
- net RSSI_A: now also IC1.3, R_RSSI_A.2, SJ1.1; no longer R_RSSI.2, U1.25
- net VIDOUT: no longer C2.C
Routing:
- net GND: track 118.3 -> 170.0 mm, vias 5 -> 7
- net RSSI_A_FIL: track 0.00 -> 31.2 mm, vias 0 -> 2
- net RSSI_A: track 27.7 -> 18.2 mm
- net 5V: track 82.7 -> 91.7 mm, vias 2 -> 3
- net N$6: track 29.3 -> 21.1 mm
- net CH3: track 36.7 -> 37.8 mm, vias 1 -> 3
- net VIDOUT: track 26.1 -> 25.3 mm
Other:
- board text added: "AUD"
- board text added: "CLK"
- board text added: "EN"
- board text added: "GND"
- board text added: "OPA337"
- board text added: "RSSI"
- board text added: "SDAT"
- board text added: "SSEL"
- board text added: "TS5A3359"
- board text added: "V4"
- board text added: "VCC"
- board text added: "VID"
- board text added: "bpass"
