File: pcb/base_module/rx_mod.sch (EAGLE design)
At the start: 28 parts, among them U1 ATMEGA328

Commit message: base module v4.0
Parts:
- removed C2: 470uf, SparkFun-Passives:CAP_POL7343
- added IC1: OPA336N, burr-brown:OPA336N
- added SJ1: (no value), jumper:SJ
- renumbered R_RSSI to R_RSSI_A, R_RSSI1 to R_RSSI_B
Connections:
- new net RSSI_A_FIL: IC1.-IN, IC1.OUT, SJ1.2, U1.PC2(ADC2)
- net 5V: now also IC1.V+
- net GND: now also IC1.V-
- net N$6: no longer C2.+
- net RSSI_A: now also IC1.+IN, SJ1.1; no longer U1.PC2(ADC2)
- net VIDOUT: no longer C2.-
Other:
- note added: "OPA337"
Changed lines of the file:
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@@
 <part name="GND11" library="supply1" deviceset="GND" device=""/>
 <part name="GND12" library="supply1" deviceset="GND" device=""/>
-<part name="R_RSSI" library="SparkFun" deviceset="RESISTOR" device="0603-RES" value="100K"/>
+<part name="R_RSSI_A" library="SparkFun" deviceset="RESISTOR" device="0603-RES" value="100K"/>
 <part name="R_SPI_SEL" library="rcl" deviceset="R-US_" device="R0805" value="10K"/>
 <part name="R_SPIDATA" library="rcl" deviceset="R-US_" device="R0805" value="10K"/>
@@
 <part name="U$1" library="#fpv" deviceset="SMA_ANTENNA" device=""/>
 <part name="C1" library="SparkFun-Passives" deviceset="CAP_POL" device="7343" value="470uf"/>
-<part name="C2" library="SparkFun-Passives" deviceset="CAP_POL" device="7343" value="470uf"/>
 <part name="P+8" library="SparkFun" deviceset="3.3V" device="" value="VCC"/>
 <part name="GND16" library="supply1" deviceset="GND" device=""/>
@@
 <part name="GND3" library="supply1" deviceset="GND" device=""/>
 <part name="P+2" library="SparkFun" deviceset="3.3V" device="" value="VCC"/>
-<part name="R_RSSI1" library="SparkFun" deviceset="RESISTOR" device="0603-RES" value="100K"/>
+<part name="R_RSSI_B" library="SparkFun" deviceset="RESISTOR" device="0603-RES" value="100K"/>
 <part name="U2" library="ts5a3359" deviceset="TS5A3359" device=""/>
 <part name="JP4" library="SparkFun-Connectors" deviceset="M04" device="PTH"/>
@@
 <part name="C3" library="adafruit" deviceset="C-US" device="C0603" value="0.1uf"/>
 <part name="GND18" library="supply1" deviceset="GND" device=""/>
+<part name="IC1" library="burr-brown" deviceset="OPA336" device="N"/>
+<part name="GND19" library="supply1" deviceset="GND" device=""/>
+<part name="P+5" library="SparkFun" deviceset="3.3V" device="" value="VCC"/>
+<part name="SJ1" library="jumper" deviceset="SJ" device=""/>
 </parts>
 <sheets>
@@
 <text x="213.36" y="88.9" size="3.81" layer="95">RECEIVER 1</text>
 <text x="114.3" y="119.38" size="3.81" layer="95">FTDI</text>
+<text x="20.32" y="142.24" size="1.778" layer="95">OPA337</text>
 </plain>
 <instances>
@@
 <instance part="GND11" gate="1" x="200.66" y="40.64"/>
 <instance part="GND12" gate="1" x="68.58" y="121.92"/>
-<instance part="R_RSSI" gate="G$1" x="274.32" y="68.58" rot="R180"/>
+<instance part="R_RSSI_A" gate="G$1" x="274.32" y="68.58" rot="R180"/>
 <instance part="R_SPI_SEL" gate="G$1" x="119.38" y="33.02"/>
 <instance part="R_SPIDATA" gate="G$1" x="119.38" y="30.48"/>
@@
 <instance part="U$1" gate="G$1" x="170.18" y="35.56"/>
 <instance part="C1" gate="G$1" x="195.58" y="78.74"/>
-<instance part="C2" gate="G$1" x="213.36" y="127" rot="R90"/>
 <instance part="P+8" gate="G$1" x="195.58" y="83.82"/>
 <instance part="GND16" gate="1" x="195.58" y="63.5"/>
@@
 <instance part="GND3" gate="1" x="172.72" y="104.14"/>
 <instance part="P+2" gate="G$1" x="208.28" y="134.62"/>
-<instance part="R_RSSI1" gate="G$1" x="152.4" y="154.94" rot="R180"/>
+<instance part="R_RSSI_B" gate="G$1" x="152.4" y="154.94" rot="R180"/>
 <instance part="U2" gate="G$1" x="190.5" y="121.92"/>
 <instance part="JP4" gate="G$1" x="238.76" y="147.32"/>
@@
 <instance part="C3" gate="G$1" x="210.82" y="132.08" rot="R90"/>
 <instance part="GND18" gate="1" x="218.44" y="132.08" rot="R90"/>
+<instance part="IC1" gate="G$1" x="17.78" y="147.32" smashed="yes">
+<attribute name="NAME" x="20.32" y="153.035" size="1.778" layer="95"/>
+</instance>
+<instance part="GND19" gate="1" x="15.24" y="134.62"/>
+<instance part="P+5" gate="G$1" x="15.24" y="157.48"/>
+<instance part="SJ1" gate="1" x="10.16" y="114.3"/>
 </instances>
 <busses>
@@
 <wire x1="279.4" y1="68.58" x2="281.94" y2="68.58" width="0.1524" layer="91"/>
 <wire x1="281.94" y1="68.58" x2="281.94" y2="63.5" width="0.1524" layer="91"/>
-<pinref part="R_RSSI" gate="G$1" pin="1"/>
+<pinref part="R_RSSI_A" gate="G$1" pin="1"/>
 </segment>
 <segment>
@@
 <pinref part="JP3" gate="G$1" pin="6"/>
 <junction x="134.62" y="157.48"/>
-<pinref part="R_RSSI1" gate="G$1" pin="1"/>
+<pinref part="R_RSSI_B" gate="G$1" pin="1"/>
 <junction x="157.48" y="152.4"/>
 <wire x1="157.48" y1="152.4" x2="157.48" y2="154.94" width="0.1524" layer="91"/>
@@
 <pinref part="GND18" gate="1" pin="GND"/>
 </segment>
+<segment>
+<pinref part="IC1" gate="G$1" pin="V-"/>
+<wire x1="15.24" y1="139.7" x2="15.24" y2="137.16" width="0.1524" layer="91"/>
+<pinref part="GND19" gate="1" pin="GND"/>
+</segment>
 </net>
 <net name="TX" class="0">
@@
 <label x="256.54" y="68.58" size="1.778" layer="95"/>
 <wire x1="251.46" y1="68.58" x2="269.24" y2="68.58" width="0.1524" layer="91"/>
-<pinref part="R_RSSI" gate="G$1" pin="2"/>
+<pinref part="R_RSSI_A" gate="G$1" pin="2"/>
 <junction x="251.46" y="68.58"/>
 </segment>
 <segment>
-<pinref part="U1" gate="G$1" pin="PC2(ADC2)"/>
-<wire x1="106.68" y1="78.74" x2="111.76" y2="78.74" width="0.1524" layer="91"/>
-<label x="106.68" y="78.74" size="1.778" layer="95"/>
-<junction x="106.68" y="78.74"/>
+<pinref part="IC1" gate="G$1" pin="+IN"/>
+<wire x1="10.16" y1="149.86" x2="-7.62" y2="149.86" width="0.1524" layer="91"/>
+<label x="-7.62" y="149.86" size="1.778" layer="95"/>
+</segment>
+<segment>
+<pinref part="SJ1" gate="1" pin="1"/>
+<wire x1="5.08" y1="114.3" x2="-5.08" y2="114.3" width="0.1524" layer="91"/>
 </segment>
 </net>
@@
 <junction x="208.28" y="132.08"/>
 </segment>
+<segment>
+<pinref part="IC1" gate="G$1" pin="V+"/>
+<wire x1="15.24" y1="154.94" x2="15.24" y2="157.48" width="0.1524" layer="91"/>
+<pinref part="P+5" gate="G$1" pin="3.3V"/>
+</segment>
 </net>
 <net name="VIDOUT" class="0">
@@
 </segment>
 <segment>
-<pinref part="C2" gate="G$1" pin="-"/>
-<wire x1="218.44" y1="127" x2="226.06" y2="127" width="0.1524" layer="91"/>
-<wire x1="226.06" y1="127" x2="226.06" y2="121.92" width="0.1524" layer="91"/>
 <pinref part="R_VIDOUT" gate="G$1" pin="2"/>
 <wire x1="226.06" y1="121.92" x2="226.06" y2="119.38" width="0.1524" layer="91"/>
 <wire x1="226.06" y1="119.38" x2="220.98" y2="119.38" width="0.1524" layer="91"/>
 <wire x1="226.06" y1="121.92" x2="236.22" y2="121.92" width="0.1524" layer="91"/>
-<junction x="226.06" y="121.92"/>
 <label x="231.14" y="121.92" size="1.778" layer="95"/>
 </segment>
@@
 <label x="134.62" y="154.94" size="1.778" layer="95"/>
 <junction x="134.62" y="154.94"/>
-<pinref part="R_RSSI1" gate="G$1" pin="2"/>
+<pinref part="R_RSSI_B" gate="G$1" pin="2"/>
 </segment>
 <segment>
@@
 <net name="N$6" class="0">
 <segment>
-<pinref part="C2" gate="G$1" pin="+"/>
-<wire x1="210.82" y1="127" x2="208.28" y2="127" width="0.1524" layer="91"/>
-<wire x1="208.28" y1="127" x2="208.28" y2="121.92" width="0.1524" layer="91"/>
 <pinref part="R_VIDOUT" gate="G$1" pin="1"/>
 <wire x1="208.28" y1="121.92" x2="208.28" y2="119.38" width="0.1524" layer="91"/>
 <wire x1="208.28" y1="119.38" x2="210.82" y2="119.38" width="0.1524" layer="91"/>
 <wire x1="203.2" y1="121.92" x2="208.28" y2="121.92" width="0.1524" layer="91"/>
-<junction x="208.28" y="121.92"/>
 <pinref part="U2" gate="G$1" pin="COM"/>
 <junction x="203.2" y="121.92"/>
@@
 </segment>
 </net>
+<net name="RSSI_A_FIL" class="0">
+<segment>
+<pinref part="IC1" gate="G$1" pin="-IN"/>
+<wire x1="10.16" y1="144.78" x2="0" y2="144.78" width="0.1524" layer="91"/>
+<wire x1="0" y1="144.78" x2="0" y2="129.54" width="0.1524" layer="91"/>
+<wire x1="0" y1="129.54" x2="38.1" y2="129.54" width="0.1524" layer="91"/>
+<wire x1="38.1" y1="129.54" x2="38.1" y2="147.32" width="0.1524" layer="91"/>
+<pinref part="IC1" gate="G$1" pin="OUT"/>
+<wire x1="38.1" y1="147.32" x2="25.4" y2="147.32" width="0.1524" layer="91"/>
+<label x="27.94" y="147.32" size="1.778" layer="95"/>
+</segment>
+<segment>
+<pinref part="U1" gate="G$1" pin="PC2(ADC2)"/>
+<wire x1="106.68" y1="78.74" x2="111.76" y2="78.74" width="0.1524" layer="91"/>
+<label x="106.68" y="78.74" size="1.778" layer="95"/>
+<junction x="106.68" y="78.74"/>
+</segment>
+<segment>
+<pinref part="SJ1" gate="1" pin="2"/>
+<wire x1="15.24" y1="114.3" x2="22.86" y2="114.3" width="0.1524" layer="91"/>
+</segment>
+</net>
