File: pcb/diversity_module/div_mod.sch (EAGLE design)
At the start: 4 parts

Commit message: regulator, buffer and new SMA connetor. v1.1
Parts:
- added C1: 0.1uf, SparkFun-Capacitors:CAP0805
- added IC1: TPS77050, texas:TPS77050
- added IC2: 74AHC1G126DBV, 74xx-little-de:74AHC1G126DBV
- added JP1: POWER_JACKSLT, SparkFun-Connectors:POWER_JACKSLT
- added R2: (no value), SparkFun-Passives:RESISTOR0805-RES
- added R3: 10k, SparkFun-Passives:RESISTOR0805-RES
- added SJ2: (no value), jumper:SJ
- added STATUS: (no value), led:LEDCHIP-LED0805
- added U$3: EB-85ASMD, SparkFun-Connectors:EB-85ASMD
Connections:
- new net ENABLE: IC1.!EN, IC2A.OE, JP3.7, R3.2, U$3.PPS
- new net N$2: R2.1, STATUS.A
- new net RSSI_MOD: IC2A.I, RECEIVER_A.RSSI, SJ2.1
- new net VIN_UNREG: IC1.IN, JP1.PWR
- net 5V: now also C1.1, IC1.OUT, IC2P.VCC, R2.2; no longer JP3.7
- net GND: now also C1.2, IC1.GND, IC2P.GND, JP1.GND, JP1.GNDBREAK, R3.1, STATUS.C, U$3.RX2
- net RSSI_B: now also IC2A.O, SJ2.2, U$3.TX2; no longer RECEIVER_A.RSSI
- net RXVIDOUT2: now also U$3.RX1
- net SPI_CLK: now also U$3.TX1
- net SPI_DATA: now also U$3.VCC
- net SPI_SEL_B: now also U$3.GND
Other:
- note added: "buffer bypass"
- moved on the sheet: JP3

Commit message: LDO name replaced
Parts:
- IC1: value TPS77050 -> REG113; device texas:TPS77050 -> texas:REG113
Connections:
- net ENABLE: now also IC1.EN; no longer IC1.!EN
Changed lines of the file:
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@@
 <part name="R1" library="SparkFun-Passives" deviceset="RESISTOR" device="0805-RES"/>
 <part name="IC2" library="74xx-little-de" deviceset="74*1G126" device="DBV" technology="AHC" value="74AHC1G126DBV"/>
-<part name="IC1" library="texas" deviceset="TPS770*" device="" technology="50"/>
+<part name="IC1" library="texas" deviceset="REG113" device=""/>
 <part name="SJ2" library="jumper" deviceset="SJ" device=""/>
 <part name="JP1" library="SparkFun-Connectors" deviceset="POWER_JACK" device="SLT"/>
@@
 </segment>
 <segment>
-<pinref part="IC1" gate="G$1" pin="!EN"/>
+<pinref part="IC1" gate="G$1" pin="EN"/>
 <wire x1="228.6" y1="147.32" x2="215.9" y2="147.32" width="0.1524" layer="91"/>
 <label x="210.82" y="147.32" size="1.778" layer="95"/>

Commit message: diversity module v2.0
Parts:
- removed IC1: REG113, texas:REG113
- removed IC2: 74AHC1G126DBV, 74xx-little-de:74AHC1G126DBV
- added C2: 1uf, SparkFun-Capacitors:CAP0805
- added IC3: OPA336N, burr-brown:OPA336N
- added JP2: (no value), SparkFun-Connectors:M02LOCK
- added SJ1: (no value), jumper:SJ
- added V1: LP38692P, lp38692:LP38692P
- C1: value 0.1uf -> 1uf
- JP1: value POWER_JACKSLT -> 5.5x2.1mm Barrel; device SparkFun-Connectors:POWER_JACKSLT -> SparkFun-Connectors:POWER_JACKSMD
- renumbered STATUS to STAT
Connections:
- net 5V: now also IC3.V+, SJ1.2, V1.VOUT; no longer IC1.OUT, IC2P.VCC
- net ENABLE: now also SJ1.1, V1.EN; no longer IC1.EN, IC2A.OE
- net GND: now also C2.2, IC3.V-, JP2.1, V1.GND; no longer IC1.GND, IC2P.GND
- net RSSI_B: now also IC3.-IN, IC3.OUT; no longer IC2A.O
- net RSSI_MOD: now also IC3.+IN; no longer IC2A.I
- net VIN_UNREG: now also C2.1, JP2.2, V1.IN; no longer IC1.IN
Other:
- note added: "OPA337"
- note added: "power"
- moved on the sheet: JP1, SJ2

Commit message: diversity board v2.1
Parts:
- added R4: 100k, SparkFun-Passives:RESISTOR0805-RES
Connections:
- new net ENABLE_P: JP3.7, R4.2, SJ1.1, U$3.PPS
- net ENABLE: now also R4.1; no longer JP3.7, SJ1.1, U$3.PPS
Other:
- moved on the sheet: C2, R3
Changed lines of the file:
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@@
 <part name="SJ1" library="jumper" deviceset="SJ" device=""/>
 <part name="P+1" library="SparkFun" deviceset="3.3V" device="" value="VCC"/>
+<part name="R4" library="SparkFun-Passives" deviceset="RESISTOR" device="0805-RES" value="100k"/>
 </parts>
 <sheets>
@@
 <instance part="P+3" gate="G$1" x="284.48" y="157.48"/>
 <instance part="GND6" gate="1" x="284.48" y="121.92"/>
-<instance part="R3" gate="G$1" x="215.9" y="142.24" rot="R90"/>
-<instance part="GND7" gate="1" x="215.9" y="132.08"/>
+<instance part="R3" gate="G$1" x="220.98" y="142.24" rot="R90"/>
+<instance part="GND7" gate="1" x="220.98" y="132.08"/>
 <instance part="IC3" gate="G$1" x="116.84" y="83.82" smashed="yes">
 <attribute name="NAME" x="119.38" y="89.535" size="1.778" layer="95"/>
@@
 <instance part="P+5" gate="G$1" x="114.3" y="93.98"/>
 <instance part="V1" gate="G$1" x="241.3" y="147.32"/>
-<instance part="C2" gate="G$1" x="203.2" y="142.24"/>
-<instance part="GND2" gate="1" x="203.2" y="132.08"/>
+<instance part="C2" gate="G$1" x="190.5" y="142.24"/>
+<instance part="GND2" gate="1" x="190.5" y="132.08"/>
 <instance part="JP2" gate="G$1" x="162.56" y="91.44"/>
 <instance part="GND12" gate="1" x="182.88" y="86.36"/>
 <instance part="SJ1" gate="1" x="114.3" y="43.18"/>
 <instance part="P+1" gate="G$1" x="134.62" y="48.26"/>
+<instance part="R4" gate="G$1" x="213.36" y="147.32" rot="R180"/>
 </instances>
 <busses>
@@
 <pinref part="R3" gate="G$1" pin="1"/>
 <pinref part="GND7" gate="1" pin="GND"/>
-<wire x1="215.9" y1="134.62" x2="215.9" y2="137.16" width="0.1524" layer="91"/>
+<wire x1="220.98" y1="134.62" x2="220.98" y2="137.16" width="0.1524" layer="91"/>
 </segment>
 <segment>
@@
 <pinref part="GND2" gate="1" pin="GND"/>
 <pinref part="C2" gate="G$1" pin="2"/>
-<wire x1="203.2" y1="134.62" x2="203.2" y2="139.7" width="0.1524" layer="91"/>
+<wire x1="190.5" y1="134.62" x2="190.5" y2="139.7" width="0.1524" layer="91"/>
 </segment>
 <segment>
@@
 <net name="ENABLE" class="0">
 <segment>
+<wire x1="226.06" y1="147.32" x2="220.98" y2="147.32" width="0.1524" layer="91"/>
+<pinref part="R3" gate="G$1" pin="2"/>
+<pinref part="V1" gate="G$1" pin="EN"/>
+<junction x="226.06" y="147.32"/>
+<pinref part="R4" gate="G$1" pin="1"/>
+<wire x1="218.44" y1="147.32" x2="220.98" y2="147.32" width="0.1524" layer="91"/>
+<junction x="220.98" y="147.32"/>
+</segment>
+</net>
+<net name="RSSI_MOD" class="0">
+<segment>
+<pinref part="RECEIVER_A" gate="G$1" pin="RSSI"/>
+<label x="256.54" y="68.58" size="1.778" layer="95"/>
+<wire x1="251.46" y1="68.58" x2="269.24" y2="68.58" width="0.1524" layer="91"/>
+<junction x="251.46" y="68.58"/>
+</segment>
+<segment>
+<pinref part="SJ2" gate="1" pin="1"/>
+<wire x1="111.76" y1="116.84" x2="96.52" y2="116.84" width="0.1524" layer="91"/>
+<label x="96.52" y="116.84" size="1.778" layer="95"/>
+<junction x="111.76" y="116.84"/>
+</segment>
+<segment>
+<pinref part="IC3" gate="G$1" pin="+IN"/>
+<wire x1="109.22" y1="86.36" x2="91.44" y2="86.36" width="0.1524" layer="91"/>
+<label x="91.44" y="86.36" size="1.778" layer="95"/>
+</segment>
+</net>
+<net name="VIN_UNREG" class="0">
+<segment>
+<pinref part="JP1" gate="G$1" pin="PWR"/>
+<wire x1="172.72" y1="116.84" x2="190.5" y2="116.84" width="0.1524" layer="91"/>
+<label x="182.88" y="116.84" size="1.778" layer="95"/>
+</segment>
+<segment>
+<wire x1="226.06" y1="152.4" x2="190.5" y2="152.4" width="0.1524" layer="91"/>
+<label x="185.42" y="152.4" size="1.778" layer="95"/>
+<pinref part="V1" gate="G$1" pin="IN"/>
+<junction x="226.06" y="152.4"/>
+<pinref part="C2" gate="G$1" pin="1"/>
+<wire x1="190.5" y1="147.32" x2="190.5" y2="152.4" width="0.1524" layer="91"/>
+<wire x1="190.5" y1="152.4" x2="187.96" y2="152.4" width="0.1524" layer="91"/>
+<junction x="190.5" y="152.4"/>
+</segment>
+<segment>
+<pinref part="JP2" gate="G$1" pin="2"/>
+<wire x1="170.18" y1="93.98" x2="182.88" y2="93.98" width="0.1524" layer="91"/>
+<label x="170.18" y="93.98" size="1.778" layer="95"/>
+</segment>
+</net>
+<net name="N$2" class="0">
+<segment>
+<pinref part="R2" gate="G$1" pin="1"/>
+<pinref part="STAT" gate="G$1" pin="A"/>
+<wire x1="284.48" y1="142.24" x2="284.48" y2="137.16" width="0.1524" layer="91"/>
+</segment>
+</net>
+<net name="ENABLE_P" class="0">
+<segment>
 <wire x1="154.94" y1="157.48" x2="170.18" y2="157.48" width="0.1524" layer="91"/>
 <pinref part="JP3" gate="G$1" pin="7"/>
@@
 </segment>
 <segment>
-<wire x1="226.06" y1="147.32" x2="215.9" y2="147.32" width="0.1524" layer="91"/>
-<label x="210.82" y="147.32" size="1.778" layer="95"/>
-<pinref part="R3" gate="G$1" pin="2"/>
-<wire x1="215.9" y1="147.32" x2="210.82" y2="147.32" width="0.1524" layer="91"/>
-<junction x="215.9" y="147.32"/>
-<pinref part="V1" gate="G$1" pin="EN"/>
-<junction x="226.06" y="147.32"/>
+<pinref part="R4" gate="G$1" pin="2"/>
+<wire x1="208.28" y1="147.32" x2="195.58" y2="147.32" width="0.1524" layer="91"/>
+<label x="195.58" y="147.32" size="1.778" layer="95"/>
 </segment>
 <segment>
@@
 </segment>
 </net>
-<net name="RSSI_MOD" class="0">
-<segment>
-<pinref part="RECEIVER_A" gate="G$1" pin="RSSI"/>
-<label x="256.54" y="68.58" size="1.778" layer="95"/>
-<wire x1="251.46" y1="68.58" x2="269.24" y2="68.58" width="0.1524" layer="91"/>
-<junction x="251.46" y="68.58"/>
-</segment>
-<segment>
-<pinref part="SJ2" gate="1" pin="1"/>
-<wire x1="111.76" y1="116.84" x2="96.52" y2="116.84" width="0.1524" layer="91"/>
-<label x="96.52" y="116.84" size="1.778" layer="95"/>
-<junction x="111.76" y="116.84"/>
-</segment>
-<segment>
-<pinref part="IC3" gate="G$1" pin="+IN"/>
-<wire x1="109.22" y1="86.36" x2="91.44" y2="86.36" width="0.1524" layer="91"/>
-<label x="91.44" y="86.36" size="1.778" layer="95"/>
-</segment>
-</net>
-<net name="VIN_UNREG" class="0">
-<segment>
-<pinref part="JP1" gate="G$1" pin="PWR"/>
-<wire x1="172.72" y1="116.84" x2="190.5" y2="116.84" width="0.1524" layer="91"/>
-<label x="182.88" y="116.84" size="1.778" layer="95"/>
-</segment>
-<segment>
-<wire x1="226.06" y1="152.4" x2="203.2" y2="152.4" width="0.1524" layer="91"/>
-<label x="193.04" y="152.4" size="1.778" layer="95"/>
-<pinref part="V1" gate="G$1" pin="IN"/>
-<junction x="226.06" y="152.4"/>
-<pinref part="C2" gate="G$1" pin="1"/>
-<wire x1="203.2" y1="147.32" x2="203.2" y2="152.4" width="0.1524" layer="91"/>
-<wire x1="203.2" y1="152.4" x2="195.58" y2="152.4" width="0.1524" layer="91"/>
-<junction x="203.2" y="152.4"/>
-</segment>
-<segment>
-<pinref part="JP2" gate="G$1" pin="2"/>
-<wire x1="170.18" y1="93.98" x2="182.88" y2="93.98" width="0.1524" layer="91"/>
-<label x="170.18" y="93.98" size="1.778" layer="95"/>
-</segment>
-</net>
-<net name="N$2" class="0">
-<segment>
-<pinref part="R2" gate="G$1" pin="1"/>
-<pinref part="STAT" gate="G$1" pin="A"/>
-<wire x1="284.48" y1="142.24" x2="284.48" y2="137.16" width="0.1524" layer="91"/>
-</segment>
-</net>

Commit message: latest from grandparents
Parts:
- removed SJ1: (no value), jumper:SJ
- JP2: device SparkFun-Connectors:M02LOCK -> SparkFun-Connectors:M02PTH
- R3: value 10k -> 100k
- R4: value 100k -> 10k
Connections:
- net 5V: no longer SJ1.2
- net ENABLE_P: no longer SJ1.1
Other:
- note removed: "power"
Changed lines of the file:
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@@
 <?xml version="1.0" encoding="utf-8"?>
 <!DOCTYPE eagle SYSTEM "eagle.dtd">
-<eagle version="7.5.0">
+<eagle version="7.7.0">
 <drawing>
 <settings>
@@
 <part name="P+3" library="SparkFun" deviceset="3.3V" device="" value="VCC"/>
 <part name="GND6" library="supply1" deviceset="GND" device=""/>
-<part name="R3" library="SparkFun-Passives" deviceset="RESISTOR" device="0805-RES" value="10k"/>
+<part name="R3" library="SparkFun-Passives" deviceset="RESISTOR" device="0805-RES" value="100k"/>
 <part name="GND7" library="supply1" deviceset="GND" device=""/>
 <part name="IC3" library="burr-brown" deviceset="OPA336" device="N"/>
@@
 <part name="C2" library="SparkFun-Capacitors" deviceset="CAP" device="0805" value="1uf"/>
 <part name="GND2" library="supply1" deviceset="GND" device=""/>
-<part name="JP2" library="SparkFun-Connectors" deviceset="M02" device="LOCK"/>
+<part name="JP2" library="SparkFun-Connectors" deviceset="M02" device="PTH"/>
 <part name="GND12" library="supply1" deviceset="GND" device=""/>
-<part name="SJ1" library="jumper" deviceset="SJ" device=""/>
-<part name="P+1" library="SparkFun" deviceset="3.3V" device="" value="VCC"/>
-<part name="R4" library="SparkFun-Passives" deviceset="RESISTOR" device="0805-RES" value="100k"/>
+<part name="R4" library="SparkFun-Passives" deviceset="RESISTOR" device="0805-RES" value="10k"/>
 </parts>
 <sheets>
@@
 <text x="111.76" y="111.76" size="1.778" layer="97">buffer bypass</text>
 <text x="119.38" y="78.74" size="1.778" layer="95">OPA337</text>
-<text x="106.68" y="38.1" size="1.778" layer="97">power</text>
 </plain>
 <instances>
@@
 <instance part="JP2" gate="G$1" x="162.56" y="91.44"/>
 <instance part="GND12" gate="1" x="182.88" y="86.36"/>
-<instance part="SJ1" gate="1" x="114.3" y="43.18"/>
-<instance part="P+1" gate="G$1" x="134.62" y="48.26"/>
 <instance part="R4" gate="G$1" x="213.36" y="147.32" rot="R180"/>
 </instances>
@@
 <pinref part="P+5" gate="G$1" pin="3.3V"/>
 </segment>
-<segment>
-<pinref part="SJ1" gate="1" pin="2"/>
-<wire x1="119.38" y1="43.18" x2="134.62" y2="43.18" width="0.1524" layer="91"/>
-<pinref part="P+1" gate="G$1" pin="3.3V"/>
-<wire x1="134.62" y1="43.18" x2="134.62" y2="48.26" width="0.1524" layer="91"/>
-</segment>
 </net>
 <net name="AUDOUT" class="0">
@@
 <label x="195.58" y="147.32" size="1.778" layer="95"/>
 </segment>
-<segment>
-<pinref part="SJ1" gate="1" pin="1"/>
-<wire x1="109.22" y1="43.18" x2="88.9" y2="43.18" width="0.1524" layer="91"/>
-<label x="93.98" y="43.18" size="1.778" layer="95"/>
-</segment>
-</net>
+</net>
